File: board/kicad/USB_UART_Converter_ch32x033/USB_UART_Converter_ch32x033.kicad_pcb (KiCad board)
At the start: 4 copper layers, 82 x 57.7 mm, 9 parts, among them J2 PRG, J3 U1, J4 I2C, J5 SPI, J7 USB_C_Receptacle_USB2.0_16P, SW2 SW_SPDT, U3 HT75xx-1-SOT89

Commit message: README, img
Other:
- board size 82 x 57.7 mm -> 24.9 x 20 mm
Changed lines of the file:
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@@
 			(at -2.54 5.65 0)
 			(layer "F.Fab")
+			(hide yes)
 			(effects
 				(font
@@
 	)
 	(gr_line
-		(start 191.48 97.01)
+		(start 134.495948 96.835652)
 		(end 109.77 96.76)
 		(stroke
@@
 	)
 	(gr_line
-		(start 109.77 39.28)
-		(end 191.73 39.28)
+		(start 109.9 76.9)
+		(end 134.7 76.8)
 		(stroke
 			(width 0.05)
@@
 	)
 	(gr_line
-		(start 191.73 39.28)
-		(end 191.48 97.01)
+		(start 134.7 76.8)
+		(end 134.495948 96.835688)
 		(stroke
 			(width 0.05)
@@
 	(gr_line
 		(start 109.77 96.76)
-		(end 109.77 39.28)
+		(end 109.9 76.9)
 		(stroke
 			(width 0.05)
@@
 	)
 	(gr_text "SPI"
-		(at 127.2 81 0)
+		(at 127.3 81.5 0)
 		(layer "F.SilkS")
 		(effects
@@
 	)
 	(gr_text "I2C"
-		(at 127.7 92.8 0)
+		(at 127.6 92.5 0)
 		(layer "F.SilkS")
 		(effects
