File: board/kicad/USB_UART_Converter_ch32x033/USB_UART_Converter_ch32x033.kicad_sch (KiCad schematic)
At the start: 11 parts, among them J2 PRG, J3 U1, J4 I2C, J5 SPI, J7 USB_C_Receptacle_USB2.0_16P, SW1 SW_Omron_B3FS, SW2 SW_SPDT, U3 HT75xx-1-SOT89

Commit message: README, img
Other:
- company: (none) -> svddevelop
- title: (none) -> CDC_UAERT_SPI_I2C_Converter3
Changed lines of the file:
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@@
 	(generator_version "9.0")
 	(paper "A4")
+	(title_block
+		(title "CDC_UAERT_SPI_I2C_Converter3")
+		(company "svddevelop")
+	)
 	(junction
 		(at 198.12 43.18)
